Commit message: cx110l is good now. URDF will simulate using the CX110l joints and links; need to adjust limits yet. also need to build cx165l model (copy/paste/edit)

File: cx110l/urdf/cx110l_description.urdf.xacro (robot description, xacro)
@@ -9,5 +9,5 @@
       rpy_offset="0 0 0"
       mesh_package="khi2cpp_hw_description/cx110l"
-      mesh_name="link_0"
+      mesh_name="cx165l-base"
   />
   <xacro:create_link
@@ -16,5 +16,5 @@
       rpy_offset="0 0 0"
       mesh_package="khi2cpp_hw_description/cx110l"
-      mesh_name="link_1"
+      mesh_name="cx165l-j1"
   />
   <xacro:create_link
@@ -23,5 +23,5 @@
       rpy_offset="0 0 0"
       mesh_package="khi2cpp_hw_description/cx110l"
-      mesh_name="link_2"
+      mesh_name="cx165l-j2"
   />
   <xacro:create_link
@@ -30,5 +30,5 @@
       rpy_offset="0 0 0"
       mesh_package="khi2cpp_hw_description/cx110l"
-      mesh_name="link_3"
+      mesh_name="cx165l-j3"
   />
   <xacro:create_link
@@ -37,5 +37,5 @@
       rpy_offset="0 0 0"
       mesh_package="khi2cpp_hw_description/cx110l"
-      mesh_name="link_4"
+      mesh_name="cx165l-j4"
   />
   <xacro:create_link
@@ -44,5 +44,5 @@
       rpy_offset="0 0 0"
       mesh_package="khi2cpp_hw_description/cx110l"
-      mesh_name="link_5"
+      mesh_name="cx165l-j5"
   />
   <xacro:create_link
@@ -51,7 +51,13 @@
       rpy_offset="0 0 0"
       mesh_package="khi2cpp_hw_description/cx110l"
-      mesh_name="link_6"
+      mesh_name="cx165l-j6"
   />
-  <link name="ft_frame"/>
+  <xacro:create_link
+      link_name="pushcorp"
+      xyz_offset="0 0 0"
+      rpy_offset="0 0 0"
+      mesh_package="khi2cpp_hw_description/cx110l"
+      mesh_name="cx165l-pushcorp"
+  />
   <link name="tool0"/>
   <!-- base_joint fixes base_link to the environment -->
@@ -60,5 +66,5 @@
     <child link="base_link"/>
     <origin xyz="0 0 0" rpy="0 0 0"/>
-    <axis xyz="0 0 1"/>
+    <axis xyz="0 0 -1"/>
   </joint>
   <!-- joints - main serial chain -->
@@ -66,6 +72,6 @@
     <parent link="base_link"/>
     <child link="link_1"/>
-    <origin xyz="0 0 0.061584" rpy="0 0 0"/>
-    <axis xyz="0 0 1"/>
+    <origin xyz="0 0 0.55" rpy="0 0 0"/>
+    <axis xyz="0 0 -1"/>
     <limit effort="1000.0" lower="${-pi}" upper="${pi}" velocity="2.5"/>
   </joint>
@@ -73,6 +79,6 @@
     <parent link="link_1"/>
     <child link="link_2"/>
-    <origin xyz="-0.101717 0 0.182284" rpy="${-pi/2} -${pi/3} ${pi/2}"/>
-    <axis xyz="0 0 1"/>
+    <origin xyz="0 0.3 0" rpy="0 0 0"/>
+    <axis xyz="1 0 0"/>
     <limit effort="1000.0" lower="${-pi}" upper="${pi}" velocity="2.5"/>
   </joint>
@@ -80,6 +86,6 @@
     <parent link="link_2"/>
     <child link="link_3"/>
-    <origin xyz="0.685682 0 0.041861" rpy="0 ${pi} ${pi+pi/2}"/>
-    <axis xyz="0 0 1"/>
+    <origin xyz="0 0 1.19" rpy="0 0 0" />
+    <axis xyz="1 0 0"/>
     <limit effort="1000.0" lower="${-pi}" upper="${pi}" velocity="2.5"/>
   </joint>
@@ -87,6 +93,6 @@
     <parent link="link_3"/>
     <child link="link_4"/>
-    <origin xyz="0.518777 0 0.067458" rpy="0 ${pi} ${pi+pi/6}"/>
-    <axis xyz="0 0 1"/>
+    <origin xyz="0 1.19 0.3" rpy="0 0 0" />
+    <axis xyz="0 1 0"/>
     <limit effort="1000.0" lower="${-pi}" upper="${pi}" velocity="2.5"/>
   </joint>
@@ -94,6 +100,6 @@
     <parent link="link_4"/>
     <child link="link_5"/>
-    <origin xyz="0.112654 0 0.110903" rpy="${pi/2} ${pi} ${pi/2}"/>
-    <axis xyz="0 0 1"/>
+    <origin xyz="0 0 0" rpy="0 0 0"/>
+    <axis xyz="1 0 0"/>
     <limit effort="1000.0" lower="${-pi}" upper="${pi}" velocity="2.5"/>
   </joint>
@@ -101,15 +107,15 @@
     <parent link="link_5"/>
     <child link="link_6"/>
-    <origin xyz="-0.085976 0 0.133436" rpy="0 ${-pi/2} 0"/>
-    <axis xyz="0 0 1"/>
+    <origin xyz="0 0.235 0" rpy="0 0 0" />
+    <axis xyz="0 1 0"/>
     <limit effort="1000.0" lower="${-pi}" upper="${pi}" velocity="2.5"/>
   </joint>
-  <joint name="joint-ft_frame" type="fixed">
+  <joint name="pushcorp" type="fixed">
     <parent link="link_6"/>
-    <child link="ft_frame"/>
-    <origin xyz="0 0 0" rpy="0 0 0"/>
+    <child link="pushcorp"/>
+      <origin xyz="0 0.0949325000000025 0" rpy="0 1.5707963267949 0" />
   </joint>
   <joint name="joint-tool" type="fixed">
-    <parent link="ft_frame"/>
+    <parent link="pushcorp"/>
     <child link="tool0"/>
     <origin xyz="0 0 .185" rpy="0 0 0"/>

Commit message: isu lab urdf added

File: cx110l/urdf/cx110l_description.urdf.xacro (robot description, xacro)
@@ -2,4 +2,34 @@
 <robot xmlns:xacro="http://www.ros.org/wiki/xacro">
   <xacro:macro name="cx110l_description">
+  <!-- link mass [kg] -->
+  <!-- CURRENTLY ESIMATES - NEED DATA FROM KAWASAKI -->
+  <xacro:property name="j0_mass" value="310"/>
+  <xacro:property name="j1_mass" value="526"/>
+  <xacro:property name="j2_mass" value="9"/>
+  <xacro:property name="j3_mass" value="66"/>
+  <xacro:property name="j4_mass" value="109"/>
+  <xacro:property name="j5_mass" value="72"/>
+  <xacro:property name="j6_mass" value="3"/>
+  <xacro:property name="pushcorp_mass" value="30"/>
+  <!-- joint limits [rad] -->
+  <xacro:property name="j1_lower_limit" value="${radians(-160)}"/>
+  <xacro:property name="j1_upper_limit" value="${radians( 160)}"/>
+  <xacro:property name="j2_lower_limit" value="${radians(-60)}"/>
+  <xacro:property name="j2_upper_limit" value="${radians( 80)}"/>
+  <xacro:property name="j3_lower_limit" value="${radians(-75)}"/>
+  <xacro:property name="j3_upper_limit" value="${radians( 95)}"/>
+  <xacro:property name="j4_lower_limit" value="${radians(-210)}"/>
+  <xacro:property name="j4_upper_limit" value="${radians( 210)}"/>
+  <xacro:property name="j5_lower_limit" value="${radians(-120)}"/>
+  <xacro:property name="j5_upper_limit" value="${radians( 120)}"/>
+  <xacro:property name="j6_lower_limit" value="${radians(-360)}"/>
+  <xacro:property name="j6_upper_limit" value="${radians( 360)}"/>
+  <!-- joint velocity limits [rad/s] -->
+  <xacro:property name="j1_velocity_limit" value="${radians(130)}"/>
+  <xacro:property name="j2_velocity_limit" value="${radians(125)}"/>
+  <xacro:property name="j3_velocity_limit" value="${radians(125)}"/>
+  <xacro:property name="j4_velocity_limit" value="${radians(180)}"/>
+  <xacro:property name="j5_velocity_limit" value="${radians(180)}"/>
+  <xacro:property name="j6_velocity_limit" value="${radians(280)}"/>
   <!-- helper macro -->
   <xacro:include filename="$(find khi2cpp_hw_description)/cx110l/urdf/inc/create_link.xacro"/>
@@ -10,4 +40,5 @@
       mesh_package="khi2cpp_hw_description/cx110l"
       mesh_name="cx165l-base"
+      link_mass = "${j0_mass}"
   />
   <xacro:create_link
@@ -17,4 +48,5 @@
       mesh_package="khi2cpp_hw_description/cx110l"
       mesh_name="cx165l-j1"
+      link_mass = "${j1_mass}"
   />
   <xacro:create_link
@@ -24,4 +56,5 @@
       mesh_package="khi2cpp_hw_description/cx110l"
       mesh_name="cx165l-j2"
+      link_mass = "${j2_mass}"
   />
   <xacro:create_link
@@ -31,4 +64,5 @@
       mesh_package="khi2cpp_hw_description/cx110l"
       mesh_name="cx165l-j3"
+      link_mass = "${j3_mass}"
   />
   <xacro:create_link
@@ -38,4 +72,5 @@
       mesh_package="khi2cpp_hw_description/cx110l"
       mesh_name="cx165l-j4"
+      link_mass = "${j4_mass}"
   />
   <xacro:create_link
@@ -45,4 +80,5 @@
       mesh_package="khi2cpp_hw_description/cx110l"
       mesh_name="cx165l-j5"
+      link_mass = "${j5_mass}"
   />
   <xacro:create_link
@@ -52,4 +88,5 @@
       mesh_package="khi2cpp_hw_description/cx110l"
       mesh_name="cx165l-j6"
+      link_mass = "${j6_mass}"
   />
   <xacro:create_link
@@ -59,4 +96,5 @@
       mesh_package="khi2cpp_hw_description/cx110l"
       mesh_name="cx165l-pushcorp"
+      link_mass = "${pushcorp_mass}"
   />
   <link name="tool0"/>
@@ -65,5 +103,5 @@
     <parent link="world"/>
     <child link="base_link"/>
-    <origin xyz="0 0 0" rpy="0 0 0"/>
+    <origin xyz="0 0 0.0254" rpy="0 0 0"/>
     <axis xyz="0 0 -1"/>
   </joint>
@@ -74,5 +112,5 @@
     <origin xyz="0 0 0.55" rpy="0 0 0"/>
     <axis xyz="0 0 -1"/>
-    <limit effort="1000.0" lower="${-pi}" upper="${pi}" velocity="2.5"/>
+    <limit effort="1000.0" lower="${j1_lower_limit}" upper="${j1_upper_limit}" velocity="${j1_velocity_limit}"/>
   </joint>
   <joint name="joint_2" type="revolute">
@@ -81,5 +119,5 @@
     <origin xyz="0 0.3 0" rpy="0 0 0"/>
     <axis xyz="1 0 0"/>
-    <limit effort="1000.0" lower="${-pi}" upper="${pi}" velocity="2.5"/>
+    <limit effort="1000.0" lower="${j2_lower_limit}" upper="${j2_upper_limit}" velocity="${j2_velocity_limit}"/>
   </joint>
   <joint name="joint_3" type="revolute">
@@ -88,5 +126,5 @@
     <origin xyz="0 0 1.19" rpy="0 0 0" />
     <axis xyz="1 0 0"/>
-    <limit effort="1000.0" lower="${-pi}" upper="${pi}" velocity="2.5"/>
+    <limit effort="1000.0" lower="${j3_lower_limit}" upper="${j3_upper_limit}" velocity="${j3_velocity_limit}"/>
   </joint>
   <joint name="joint_4" type="revolute">
@@ -95,5 +133,5 @@
     <origin xyz="0 1.19 0.3" rpy="0 0 0" />
     <axis xyz="0 1 0"/>
-    <limit effort="1000.0" lower="${-pi}" upper="${pi}" velocity="2.5"/>
+    <limit effort="1000.0" lower="${j4_lower_limit}" upper="${j4_upper_limit}" velocity="${j4_velocity_limit}"/>
   </joint>
   <joint name="joint_5" type="revolute">
@@ -102,5 +140,5 @@
     <origin xyz="0 0 0" rpy="0 0 0"/>
     <axis xyz="1 0 0"/>
-    <limit effort="1000.0" lower="${-pi}" upper="${pi}" velocity="2.5"/>
+    <limit effort="1000.0" lower="${j5_lower_limit}" upper="${j5_upper_limit}" velocity="${j5_velocity_limit}"/>
   </joint>
   <joint name="joint_6" type="revolute">
@@ -109,5 +147,5 @@
     <origin xyz="0 0.235 0" rpy="0 0 0" />
     <axis xyz="0 1 0"/>
-    <limit effort="1000.0" lower="${-pi}" upper="${pi}" velocity="2.5"/>
+    <limit effort="1000.0" lower="${j6_lower_limit}" upper="${j6_upper_limit}" velocity="${j6_velocity_limit}"/>
   </joint>
   <joint name="pushcorp" type="fixed">

File: cx110l/urdf/inc/create_link.xacro (robot description, xacro)
@@ -1,4 +1,11 @@
 <?xml version="1.0"?>
 <robot xmlns:xacro="http://wiki.ros.org/xacro">
+  <!-- inertial macro - assign intertial properties to links-->
+  <xacro:macro name="default_inertial" params="mass">
+    <inertial>
+      <mass value="${mass}" />
+      <inertia ixx="0.1" ixy="0.0" ixz="0.0" iyy="0.1" iyz="0.0" izz="0.1" />
+    </inertial>
+  </xacro:macro>
   <xacro:macro name="create_link" params="
         link_name
@@ -6,5 +13,7 @@
         rpy_offset
         mesh_package
-        mesh_name">
+        mesh_name
+        link_mass
+        ">
     <link name="${link_name}">
       <visual>
@@ -13,4 +22,8 @@
           <mesh filename="package://${mesh_package}/meshes/visual/${mesh_name}.dae"/>
         </geometry>
+        <material
+          name="">
+          <color rgba="0.75294 0.75294 0.75294 1" />
+        </material>
       </visual>
       <collision>
@@ -20,8 +33,5 @@
         </geometry>
       </collision>
-      <inertial>
-        <mass value="1"/>
-        <inertia ixx="1.0" ixy="0.0" ixz="0.0" iyy="1.0" iyz="0.0" izz="1.0"/>
-      </inertial>
+      <xacro:default_inertial mass="${link_mass}"/>
     </link>
   </xacro:macro>

Commit message: morning push

File: cx110l/urdf/cx110l_description.urdf.xacro (robot description, xacro)
@@ -13,10 +13,10 @@
   <xacro:property name="pushcorp_mass" value="30"/>
   <!-- joint limits [rad] -->
-  <xacro:property name="j1_lower_limit" value="${radians(-160)}"/>
-  <xacro:property name="j1_upper_limit" value="${radians( 160)}"/>
-  <xacro:property name="j2_lower_limit" value="${radians(-60)}"/>
-  <xacro:property name="j2_upper_limit" value="${radians( 80)}"/>
-  <xacro:property name="j3_lower_limit" value="${radians(-75)}"/>
-  <xacro:property name="j3_upper_limit" value="${radians( 95)}"/>
+  <xacro:property name="j1_lower_limit" value="${radians( 0 )}"/>
+  <xacro:property name="j1_upper_limit" value="${radians( 90 )}"/>
+  <xacro:property name="j2_lower_limit" value="${radians(-80 )}"/>
+  <xacro:property name="j2_upper_limit" value="${radians( 36 )}"/>
+  <xacro:property name="j3_lower_limit" value="${radians(-75 )}"/>
+  <xacro:property name="j3_upper_limit" value="${radians( 0 )}"/>
   <xacro:property name="j4_lower_limit" value="${radians(-210)}"/>
   <xacro:property name="j4_upper_limit" value="${radians( 210)}"/>
@@ -90,4 +90,5 @@
       link_mass = "${j6_mass}"
   />
+<!--
   <xacro:create_link
       link_name="pushcorp"
@@ -98,4 +99,5 @@
       link_mass = "${pushcorp_mass}"
   />
+-->
   <link name="tool0"/>
   <!-- base_joint fixes base_link to the environment -->
@@ -103,5 +105,5 @@
     <parent link="world"/>
     <child link="base_link"/>
-    <origin xyz="0 0 0.0254" rpy="0 0 0"/>
+    <origin xyz="-5.0546 0 0.0254" rpy="0 0 0"/>
     <axis xyz="0 0 -1"/>
   </joint>
@@ -149,4 +151,5 @@
     <limit effort="1000.0" lower="${j6_lower_limit}" upper="${j6_upper_limit}" velocity="${j6_velocity_limit}"/>
   </joint>
+<!--
   <joint name="pushcorp" type="fixed">
     <parent link="link_6"/>
@@ -154,8 +157,9 @@
       <origin xyz="0 0.0949325000000025 0" rpy="0 1.5707963267949 0" />
   </joint>
+-->
   <joint name="joint-tool" type="fixed">
-    <parent link="pushcorp"/>
+    <parent link="link_6"/>
     <child link="tool0"/>
-    <origin xyz="0 0 .185" rpy="0 0 0"/>
+    <origin xyz="0 0 0" rpy="0 0 0"/>
   </joint>
 </xacro:macro>

Commit message: working push

File: cx110l/urdf/cx110l_description.urdf.xacro (robot description, xacro)
@@ -32,72 +32,156 @@
   <xacro:property name="j5_velocity_limit" value="${radians(180)}"/>
   <xacro:property name="j6_velocity_limit" value="${radians(280)}"/>
-  <!-- helper macro -->
-  <xacro:include filename="$(find khi2cpp_hw_description)/cx110l/urdf/inc/create_link.xacro"/>
-  <xacro:create_link
-      link_name="base_link"
-      xyz_offset="0 0 0"
-      rpy_offset="0 0 0"
-      mesh_package="khi2cpp_hw_description/cx110l"
-      mesh_name="cx165l-base"
-      link_mass = "${j0_mass}"
-  />
-  <xacro:create_link
-      link_name="link_1"
-      xyz_offset="0 0 0"
-      rpy_offset="0 0 0"
-      mesh_package="khi2cpp_hw_description/cx110l"
-      mesh_name="cx165l-j1"
-      link_mass = "${j1_mass}"
-  />
-  <xacro:create_link
-      link_name="link_2"
-      xyz_offset="0 0 0"
-      rpy_offset="0 0 0"
-      mesh_package="khi2cpp_hw_description/cx110l"
-      mesh_name="cx165l-j2"
-      link_mass = "${j2_mass}"
-  />
-  <xacro:create_link
-      link_name="link_3"
-      xyz_offset="0 0 0"
-      rpy_offset="0 0 0"
-      mesh_package="khi2cpp_hw_description/cx110l"
-      mesh_name="cx165l-j3"
-      link_mass = "${j3_mass}"
-  />
-  <xacro:create_link
-      link_name="link_4"
-      xyz_offset="0 0 0"
-      rpy_offset="0 0 0"
-      mesh_package="khi2cpp_hw_description/cx110l"
-      mesh_name="cx165l-j4"
-      link_mass = "${j4_mass}"
-  />
-  <xacro:create_link
-      link_name="link_5"
-      xyz_offset="0 0 0"
-      rpy_offset="0 0 0"
-      mesh_package="khi2cpp_hw_description/cx110l"
-      mesh_name="cx165l-j5"
-      link_mass = "${j5_mass}"
-  />
-  <xacro:create_link
-      link_name="link_6"
-      xyz_offset="0 0 0"
-      rpy_offset="0 0 0"
-      mesh_package="khi2cpp_hw_description/cx110l"
-      mesh_name="cx165l-j6"
-      link_mass = "${j6_mass}"
-  />
-<!--
-  <xacro:create_link
-      link_name="pushcorp"
-      xyz_offset="0 0 0"
-      rpy_offset="0 0 0"
-      mesh_package="khi2cpp_hw_description/cx110l"
-      mesh_name="cx165l-pushcorp"
-      link_mass = "${pushcorp_mass}"
-  />
--->
+  <link name="base_link">
+    <visual>
+      <origin xyz="0 0 0" rpy="0 0 0"/>
+      <geometry>
+        <mesh filename="package://khi2cpp_hw_description/cx110l/meshes/visual/cx165l-base.dae"/>
+      </geometry>
+      <material
+        name="">
+        <color rgba="0.75294 0.75294 0.75294 1" />
+      </material>
+    </visual>
+    <collision>
+      <origin xyz="0 0 0" rpy="0 0 0"/>
+      <geometry>
+        <mesh filename="package://khi2cpp_hw_description/cx110l/meshes/collision/cx165l-base.stl"/>
+      </geometry>
+    </collision>
+    <xacro:default_inertial mass="${j0_mass}"/>
+  </link>
+  <link name="link_1">
+    <visual>
+      <origin xyz="0 0 0" rpy="0 0 0"/>
+      <geometry>
+        <mesh filename="package://khi2cpp_hw_description/cx110l/meshes/visual/cx165l-j1.dae"/>
+      </geometry>
+      <material
+        name="">
+        <color rgba="0.75294 0.75294 0.75294 1" />
+      </material>
+    </visual>
+    <collision>
+      <origin xyz="0 0 0" rpy="0 0 0"/>
+      <geometry>
+        <mesh filename="package://khi2cpp_hw_description/cx110l/meshes/collision/cx165l-j1.stl"/>
+      </geometry>
+    </collision>
+    <xacro:default_inertial mass="${j1_mass}"/>
+  </link>
+  <link name="link_2">
+    <visual>
+      <origin xyz="0 0 0" rpy="0 0 0"/>
+      <geometry>
+        <mesh filename="package://khi2cpp_hw_description/cx110l/meshes/visual/cx165l-j2.dae"/>
+      </geometry>
+      <material
+        name="">
+        <color rgba="0.75294 0.75294 0.75294 1" />
+      </material>
+    </visual>
+    <collision>
+      <origin xyz="0 0 0" rpy="0 0 0"/>
+      <geometry>
+        <mesh filename="package://khi2cpp_hw_description/cx110l/meshes/collision/cx165l-j2.stl"/>
+      </geometry>
+    </collision>
+    <xacro:default_inertial mass="${j2_mass}"/>
+  </link>
+  <link name="link_3">
+    <visual>
+      <origin xyz="0 0 0" rpy="0 0 0"/>
+      <geometry>
+        <mesh filename="package://khi2cpp_hw_description/cx110l/meshes/visual/cx165l-j3.dae"/>
+      </geometry>
+      <material
+        name="">
+        <color rgba="0.75294 0.75294 0.75294 1" />
+      </material>
+    </visual>
+    <collision>
+      <origin xyz="0 0 0" rpy="0 0 0"/>
+      <geometry>
+        <mesh filename="package://khi2cpp_hw_description/cx110l/meshes/collision/cx165l-j3.stl"/>
+      </geometry>
+    </collision>
+    <xacro:default_inertial mass="${j3_mass}"/>
+  </link>
+  <link name="link_4">
+    <visual>
+      <origin xyz="0 0 0" rpy="0 0 0"/>
+      <geometry>
+        <mesh filename="package://khi2cpp_hw_description/cx110l/meshes/visual/cx165l-j4.dae"/>
+      </geometry>
+      <material
+        name="">
+        <color rgba="0.75294 0.75294 0.75294 1" />
+      </material>
+    </visual>
+    <collision>
+      <origin xyz="0 0 0" rpy="0 0 0"/>
+      <geometry>
+        <mesh filename="package://khi2cpp_hw_description/cx110l/meshes/collision/cx165l-j4.stl"/>
+      </geometry>
+    </collision>
+    <xacro:default_inertial mass="${j4_mass}"/>
+  </link>
+  <link name="link_5">
+    <visual>
+      <origin xyz="0 0 0" rpy="0 0 0"/>
+      <geometry>
+        <mesh filename="package://khi2cpp_hw_description/cx110l/meshes/visual/cx165l-j5.dae"/>
+      </geometry>
+      <material
+        name="">
+        <color rgba="0.75294 0.75294 0.75294 1" />
+      </material>
+    </visual>
+    <collision>
+      <origin xyz="0 0 0" rpy="0 0 0"/>
+      <geometry>
+        <mesh filename="package://khi2cpp_hw_description/cx110l/meshes/collision/cx165l-j5.stl"/>
+      </geometry>
+    </collision>
+    <xacro:default_inertial mass="${j5_mass}"/>
+  </link>
+  <link name="link_6">
+    <visual>
+      <origin xyz="0 0 0" rpy="0 0 0"/>
+      <geometry>
+        <mesh filename="package://khi2cpp_hw_description/cx110l/meshes/visual/cx165l-j6.dae"/>
+      </geometry>
+      <material
+        name="">
+        <color rgba="0.75294 0.75294 0.75294 1" />
+      </material>
+    </visual>
+    <collision>
+      <origin xyz="0 0 0" rpy="0 0 0"/>
+      <geometry>
+        <mesh filename="package://khi2cpp_hw_description/cx110l/meshes/collision/cx165l-j6.stl"/>
+      </geometry>
+    </collision>
+    <xacro:default_inertial mass="${j6_mass}"/>
+  </link>
+  <link name="pushcorp">
+    <visual>
+      <origin xyz="0 0 0" rpy="0 0 0"/>
+      <geometry>
+        <mesh filename="package://khi2cpp_hw_description/cx110l/meshes/visual/cx165l-pushcorp.dae"/>
+      </geometry>
+      <material
+        name="">
+        <color rgba="0.75294 0.75294 0.75294 1" />
+      </material>
+    </visual>
+    <collision>
+      <origin xyz="0 0 0" rpy="0 0 0"/>
+      <geometry>
+        <mesh filename="package://khi2cpp_hw_description/cx110l/meshes/collision/cx165l-pushcorp.stl"/>
+      </geometry>
+    </collision>
+    <xacro:default_inertial mass="${pushcorp_mass}"/>
+  </link>
   <link name="tool0"/>
   <!-- base_joint fixes base_link to the environment -->
@@ -151,5 +235,4 @@
     <limit effort="1000.0" lower="${j6_lower_limit}" upper="${j6_upper_limit}" velocity="${j6_velocity_limit}"/>
   </joint>
-<!--
   <joint name="pushcorp" type="fixed">
     <parent link="link_6"/>
@@ -157,9 +240,8 @@
       <origin xyz="0 0.0949325000000025 0" rpy="0 1.5707963267949 0" />
   </joint>
--->
   <joint name="joint-tool" type="fixed">
-    <parent link="link_6"/>
+    <parent link="pushcorp"/>
     <child link="tool0"/>
-    <origin xyz="0 0 0" rpy="0 0 0"/>
+    <origin xyz="0 0 .185" rpy="0 0 0"/>
   </joint>
 </xacro:macro>

File: cx165l/urdf/cx165l_description.urdf.xacro (robot description, xacro)
@@ -13,6 +13,6 @@
   <xacro:property name="pushcorp_mass" value="30"/>
   <!-- joint limits [rad] -->
-  <xacro:property name="j1_lower_limit" value="${radians(-160)}"/>
-  <xacro:property name="j1_upper_limit" value="${radians( 160)}"/>
+  <xacro:property name="j1_lower_limit" value="${radians(-90)}"/>
+  <xacro:property name="j1_upper_limit" value="${radians( 0)}"/>
   <xacro:property name="j2_lower_limit" value="${radians(-60)}"/>
   <xacro:property name="j2_upper_limit" value="${radians( 80)}"/>
