Commit message: Updated components of driver

File: cx110l/urdf/cx110l_macro.xacro (robot description, xacro)
@@ -1,5 +1,12 @@
 <?xml version="1.0"?>
 <robot xmlns:xacro="http://www.ros.org/wiki/xacro">
-  <xacro:macro name="cx165l_description">
+  <xacro:macro name="khi_cx110l" params="prefix">
+  <!-- link rviz colors -->
+  <material name="White">
+    <color rgba="1 1 1 1"/>
+  </material>
+  <material name="Black">
+    <color rgba="0 0 0 1"/>
+  </material>
   <!-- link mass [kg] -->
   <!-- CURRENTLY ESIMATES - NEED DATA FROM KAWASAKI -->
@@ -11,12 +18,12 @@
   <xacro:property name="j5_mass" value="72"/>
   <xacro:property name="j6_mass" value="3"/>
-  <xacro:property name="pushcorp_mass" value="30"/>
+  <!-- <xacro:property name="pushcorp_mass" value="30"/> -->
   <!-- joint limits [rad] -->
-  <xacro:property name="j1_lower_limit" value="${radians(-90)}"/>
-  <xacro:property name="j1_upper_limit" value="${radians( 0)}"/>
-  <xacro:property name="j2_lower_limit" value="${radians(-60)}"/>
-  <xacro:property name="j2_upper_limit" value="${radians( 80)}"/>
-  <xacro:property name="j3_lower_limit" value="${radians(-75)}"/>
-  <xacro:property name="j3_upper_limit" value="${radians( 95)}"/>
+  <xacro:property name="j1_lower_limit" value="${radians( 0 )}"/>
+  <xacro:property name="j1_upper_limit" value="${radians( 90 )}"/>
+  <xacro:property name="j2_lower_limit" value="${radians(-80 )}"/>
+  <xacro:property name="j2_upper_limit" value="${radians( 36 )}"/>
+  <xacro:property name="j3_lower_limit" value="${radians(-75 )}"/>
+  <xacro:property name="j3_upper_limit" value="${radians( 0 )}"/>
   <xacro:property name="j4_lower_limit" value="${radians(-210)}"/>
   <xacro:property name="j4_upper_limit" value="${radians( 210)}"/>
@@ -32,216 +39,230 @@
   <xacro:property name="j5_velocity_limit" value="${radians(180)}"/>
   <xacro:property name="j6_velocity_limit" value="${radians(280)}"/>
-  <link name="base_link">
-    <visual>
-      <origin xyz="0 0 0" rpy="0 0 0"/>
-      <geometry>
-        <mesh filename="package://khi2cpp_hw_description/cx165l/meshes/visual/cx165l-base.dae"/>
-      </geometry>
-      <material
-        name="">
-        <color rgba="0.75294 0.75294 0.75294 1" />
-      </material>
-    </visual>
-    <collision>
-      <origin xyz="0 0 0" rpy="0 0 0"/>
-      <geometry>
-        <mesh filename="package://khi2cpp_hw_description/cx165l/meshes/collision/cx165l-base.stl"/>
+  <!-- link inertial(TODO : set correct link inertial )-->
+    <xacro:macro name="default_inertial" params="mass">
+      <inertial>
+        <mass value="${mass}" />
+        <inertia ixx="0.1" ixy="0.0" ixz="0.0" iyy="0.1" iyz="0.0" izz="0.1" />
+      </inertial>
+    </xacro:macro>
+    <link name="world"/>
+    <!-- Link 0 -->
+    <link name="${prefix}base_link">
+    <visual>
+      <origin
+          xyz="0 0 0"
+          rpy="0 0 0"/>
+      <geometry>
+        <mesh
+        filename="package://khi2cpp_hw_description/cx110l/meshes/visual/cx165l-base.dae"/>
+      </geometry>
+      <material
+        name="">
+        <color rgba="0.75294 0.75294 0.75294 1" />
+      </material>
+    </visual>
+    <collision>
+      <origin
+          xyz="0 0 0"
+          rpy="0 0 0"/>
+      <geometry>
+        <mesh filename="package://khi2cpp_hw_description/cx110l/meshes/collision/cx165l-base.stl"/>
       </geometry>
     </collision>
     <xacro:default_inertial mass="${j0_mass}"/>
   </link>
-  <link name="link_1">
-    <visual>
-      <origin xyz="0 0 0" rpy="0 0 0"/>
-      <geometry>
-        <mesh filename="package://khi2cpp_hw_description/cx165l/meshes/visual/cx165l-j1.dae"/>
-      </geometry>
-      <material
-        name="">
-        <color rgba="0.75294 0.75294 0.75294 1" />
-      </material>
-    </visual>
-    <collision>
-      <origin xyz="0 0 0" rpy="0 0 0"/>
-      <geometry>
-        <mesh filename="package://khi2cpp_hw_description/cx165l/meshes/collision/cx165l-j1.stl"/>
+  <link name="${prefix}link1">
+    <visual>
+      <origin xyz="0 0 0" rpy="0 0 0"/>
+      <geometry>
+        <mesh filename="package://khi2cpp_hw_description/cx110l/meshes/visual/cx165l-j1.dae"/>
+      </geometry>
+      <material
+        name="">
+        <color rgba="0.75294 0.75294 0.75294 1" />
+      </material>
+    </visual>
+    <collision>
+      <origin xyz="0 0 0" rpy="0 0 0"/>
+      <geometry>
+        <mesh filename="package://khi2cpp_hw_description/cx110l/meshes/collision/cx165l-j1.stl"/>
       </geometry>
     </collision>
     <xacro:default_inertial mass="${j1_mass}"/>
   </link>
-  <link name="link_2">
-    <visual>
-      <origin xyz="0 0 0" rpy="0 0 0"/>
-      <geometry>
-        <mesh filename="package://khi2cpp_hw_description/cx165l/meshes/visual/cx165l-j2.dae"/>
-      </geometry>
-      <material
-        name="">
-        <color rgba="0.75294 0.75294 0.75294 1" />
-      </material>
-    </visual>
-    <collision>
-      <origin xyz="0 0 0" rpy="0 0 0"/>
-      <geometry>
-        <mesh filename="package://khi2cpp_hw_description/cx165l/meshes/collision/cx165l-j2.stl"/>
+  <link name="${prefix}link2">
+    <visual>
+      <origin xyz="0 0 0" rpy="0 0 0"/>
+      <geometry>
+        <mesh filename="package://khi2cpp_hw_description/cx110l/meshes/visual/cx165l-j2.dae"/>
+      </geometry>
+      <material
+        name="">
+        <color rgba="0.75294 0.75294 0.75294 1" />
+      </material>
+    </visual>
+    <collision>
+      <origin xyz="0 0 0" rpy="0 0 0"/>
+      <geometry>
+        <mesh filename="package://khi2cpp_hw_description/cx110l/meshes/collision/cx165l-j2.stl"/>
       </geometry>
     </collision>
     <xacro:default_inertial mass="${j2_mass}"/>
   </link>
-  <link name="link_3">
-    <visual>
-      <origin xyz="0 0 0" rpy="0 0 0"/>
-      <geometry>
-        <mesh filename="package://khi2cpp_hw_description/cx165l/meshes/visual/cx165l-j3.dae"/>
-      </geometry>
-      <material
-        name="">
-        <color rgba="0.75294 0.75294 0.75294 1" />
-      </material>
-    </visual>
-    <collision>
-      <origin xyz="0 0 0" rpy="0 0 0"/>
-      <geometry>
-        <mesh filename="package://khi2cpp_hw_description/cx165l/meshes/collision/cx165l-j3.stl"/>
+  <link name="${prefix}link3">
+    <visual>
+      <origin xyz="0 0 0" rpy="0 0 0"/>
+      <geometry>
+        <mesh filename="package://khi2cpp_hw_description/cx110l/meshes/visual/cx165l-j3.dae"/>
+      </geometry>
+      <material
+        name="">
+        <color rgba="0.75294 0.75294 0.75294 1" />
+      </material>
+    </visual>
+    <collision>
+      <origin xyz="0 0 0" rpy="0 0 0"/>
+      <geometry>
+        <mesh filename="package://khi2cpp_hw_description/cx110l/meshes/collision/cx165l-j3.stl"/>
       </geometry>
     </collision>
     <xacro:default_inertial mass="${j3_mass}"/>
   </link>
-  <link name="link_4">
-    <visual>
-      <origin xyz="0 0 0" rpy="0 0 0"/>
-      <geometry>
-        <mesh filename="package://khi2cpp_hw_description/cx165l/meshes/visual/cx165l-j4.dae"/>
-      </geometry>
-      <material
-        name="">
-        <color rgba="0.75294 0.75294 0.75294 1" />
-      </material>
-    </visual>
-    <collision>
-      <origin xyz="0 0 0" rpy="0 0 0"/>
-      <geometry>
-        <mesh filename="package://khi2cpp_hw_description/cx165l/meshes/collision/cx165l-j4.stl"/>
+  <link name="${prefix}link4">
+    <visual>
+      <origin xyz="0 0 0" rpy="0 0 0"/>
+      <geometry>
+        <mesh filename="package://khi2cpp_hw_description/cx110l/meshes/visual/cx165l-j4.dae"/>
+      </geometry>
+      <material
+        name="">
+        <color rgba="0.75294 0.75294 0.75294 1" />
+      </material>
+    </visual>
+    <collision>
+      <origin xyz="0 0 0" rpy="0 0 0"/>
+      <geometry>
+        <mesh filename="package://khi2cpp_hw_description/cx110l/meshes/collision/cx165l-j4.stl"/>
       </geometry>
     </collision>
     <xacro:default_inertial mass="${j4_mass}"/>
   </link>
-  <link name="link_5">
-    <visual>
-      <origin xyz="0 0 0" rpy="0 0 0"/>
-      <geometry>
-        <mesh filename="package://khi2cpp_hw_description/cx165l/meshes/visual/cx165l-j5.dae"/>
-      </geometry>
-      <material
-        name="">
-        <color rgba="0.75294 0.75294 0.75294 1" />
-      </material>
-    </visual>
-    <collision>
-      <origin xyz="0 0 0" rpy="0 0 0"/>
-      <geometry>
-        <mesh filename="package://khi2cpp_hw_description/cx165l/meshes/collision/cx165l-j5.stl"/>
+  <link name="${prefix}link5">
+    <visual>
+      <origin xyz="0 0 0" rpy="0 0 0"/>
+      <geometry>
+        <mesh filename="package://khi2cpp_hw_description/cx110l/meshes/visual/cx165l-j5.dae"/>
+      </geometry>
+      <material
+        name="">
+        <color rgba="0.75294 0.75294 0.75294 1" />
+      </material>
+    </visual>
+    <collision>
+      <origin xyz="0 0 0" rpy="0 0 0"/>
+      <geometry>
+        <mesh filename="package://khi2cpp_hw_description/cx110l/meshes/collision/cx165l-j5.stl"/>
       </geometry>
     </collision>
     <xacro:default_inertial mass="${j5_mass}"/>
   </link>
-  <link name="link_6">
-    <visual>
-      <origin xyz="0 0 0" rpy="0 0 0"/>
-      <geometry>
-        <mesh filename="package://khi2cpp_hw_description/cx165l/meshes/visual/cx165l-j6.dae"/>
-      </geometry>
-      <material
-        name="">
-        <color rgba="0.75294 0.75294 0.75294 1" />
-      </material>
-    </visual>
-    <collision>
-      <origin xyz="0 0 0" rpy="0 0 0"/>
-      <geometry>
-        <mesh filename="package://khi2cpp_hw_description/cx165l/meshes/collision/cx165l-j6.stl"/>
+  <link name="${prefix}link6">
+    <visual>
+      <origin xyz="0 0 0" rpy="0 0 0"/>
+      <geometry>
+        <mesh filename="package://khi2cpp_hw_description/cx110l/meshes/visual/cx165l-j6.dae"/>
+      </geometry>
+      <material
+        name="">
+        <color rgba="0.75294 0.75294 0.75294 1" />
+      </material>
+    </visual>
+    <collision>
+      <origin xyz="0 0 0" rpy="0 0 0"/>
+      <geometry>
+        <mesh filename="package://khi2cpp_hw_description/cx110l/meshes/collision/cx165l-j6.stl"/>
       </geometry>
     </collision>
     <xacro:default_inertial mass="${j6_mass}"/>
   </link>
-  <link name="pushcorp">
-    <visual>
-      <origin xyz="0 0 0" rpy="0 0 0"/>
-      <geometry>
-        <mesh filename="package://khi2cpp_hw_description/cx165l/meshes/visual/cx165l-pushcorp.dae"/>
-      </geometry>
-      <material
-        name="">
-        <color rgba="0.75294 0.75294 0.75294 1" />
-      </material>
-    </visual>
-    <collision>
-      <origin xyz="0 0 0" rpy="0 0 0"/>
-      <geometry>
-        <mesh filename="package://khi2cpp_hw_description/cx165l/meshes/collision/cx165l-pushcorp.stl"/>
+  <!-- <link name="${prefix}pushcorp">
+    <visual>
+      <origin xyz="0 0 0" rpy="0 0 0"/>
+      <geometry>
+        <mesh filename="package://khi2cpp_hw_description/cx110l/meshes/visual/cx165l-pushcorp.dae"/>
+      </geometry>
+      <material
+        name="">
+        <color rgba="0.75294 0.75294 0.75294 1" />
+      </material>
+    </visual>
+    <collision>
+      <origin xyz="0 0 0" rpy="0 0 0"/>
+      <geometry>
+        <mesh filename="package://khi2cpp_hw_description/cx110l/meshes/collision/cx165l-pushcorp.stl"/>
       </geometry>
     </collision>
     <xacro:default_inertial mass="${pushcorp_mass}"/>
-  </link>
-  <link name="tool0"/>
+  </link> -->
+  <link name="${prefix}tool0"/>
   <!-- base_joint fixes base_link to the environment -->
-  <joint name="base_joint" type="fixed">
+  <joint name="${prefix}base_joint" type="fixed">
     <parent link="world"/>
-    <child link="base_link"/>
-    <origin xyz="0 0 0.0254" rpy="0 0 0"/>
+    <child link="${prefix}base_link"/>
+    <origin xyz="-5.0546 0 0.0254" rpy="0 0 0"/>
     <axis xyz="0 0 -1"/>
   </joint>
   <!-- joints - main serial chain -->
-  <joint name="joint_1" type="revolute">
-    <parent link="base_link"/>
-    <child link="link_1"/>
+  <joint name="${prefix}joint1" type="revolute">
+    <parent link="${prefix}base_link"/>
+    <child link="${prefix}link1"/>
     <origin xyz="0 0 0.55" rpy="0 0 0"/>
     <axis xyz="0 0 -1"/>
     <limit effort="1000.0" lower="${j1_lower_limit}" upper="${j1_upper_limit}" velocity="${j1_velocity_limit}"/>
   </joint>
-  <joint name="joint_2" type="revolute">
-    <parent link="link_1"/>
-    <child link="link_2"/>
+  <joint name="${prefix}joint2" type="revolute">
+    <parent link="${prefix}link1"/>
+    <child link="${prefix}link2"/>
     <origin xyz="0 0.3 0" rpy="0 0 0"/>
     <axis xyz="1 0 0"/>
     <limit effort="1000.0" lower="${j2_lower_limit}" upper="${j2_upper_limit}" velocity="${j2_velocity_limit}"/>
   </joint>
-  <joint name="joint_3" type="revolute">
-    <parent link="link_2"/>
-    <child link="link_3"/>
+  <joint name="${prefix}joint3" type="revolute">
+    <parent link="${prefix}link2"/>
+    <child link="${prefix}link3"/>
     <origin xyz="0 0 1.19" rpy="0 0 0" />
     <axis xyz="1 0 0"/>
     <limit effort="1000.0" lower="${j3_lower_limit}" upper="${j3_upper_limit}" velocity="${j3_velocity_limit}"/>
   </joint>
-  <joint name="joint_4" type="revolute">
-    <parent link="link_3"/>
-    <child link="link_4"/>
+  <joint name="${prefix}joint4" type="revolute">
+    <parent link="${prefix}link3"/>
+    <child link="${prefix}link4"/>
     <origin xyz="0 1.19 0.3" rpy="0 0 0" />
     <axis xyz="0 1 0"/>
     <limit effort="1000.0" lower="${j4_lower_limit}" upper="${j4_upper_limit}" velocity="${j4_velocity_limit}"/>
   </joint>
-  <joint name="joint_5" type="revolute">
-    <parent link="link_4"/>
-    <child link="link_5"/>
+  <joint name="${prefix}joint5" type="revolute">
+    <parent link="${prefix}link4"/>
+    <child link="${prefix}link5"/>
     <origin xyz="0 0 0" rpy="0 0 0"/>
     <axis xyz="1 0 0"/>
     <limit effort="1000.0" lower="${j5_lower_limit}" upper="${j5_upper_limit}" velocity="${j5_velocity_limit}"/>
   </joint>
-  <joint name="joint_6" type="revolute">
-    <parent link="link_5"/>
-    <child link="link_6"/>
+  <joint name="${prefix}joint6" type="revolute">
+    <parent link="${prefix}link5"/>
+    <child link="${prefix}link6"/>
     <origin xyz="0 0.235 0" rpy="0 0 0" />
     <axis xyz="0 1 0"/>
     <limit effort="1000.0" lower="${j6_lower_limit}" upper="${j6_upper_limit}" velocity="${j6_velocity_limit}"/>
   </joint>
-  <joint name="pushcorp" type="fixed">
-    <parent link="link_6"/>
-    <child link="pushcorp"/>
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