Commit message: Updated components of driver

File: cx165l/urdf/cx165l_macro.xacro (robot description, xacro)
@@ -1,5 +1,14 @@
 <?xml version="1.0"?>
 <robot xmlns:xacro="http://www.ros.org/wiki/xacro">
-  <xacro:macro name="cx110l_description">
+  <xacro:macro name="khi_cx165l" params="prefix">
+  <xacro:include filename="$(find khi2cpp_hw_description)/common/cx.transmission.xacro" />
+  <xacro:include filename="$(find khi2cpp_hw_description)/common/common.gazebo.xacro" />
+  <!-- link rviz colors -->
+  <material name="White">
+    <color rgba="1 1 1 1"/>
+  </material>
+  <material name="Black">
+    <color rgba="0 0 0 1"/>
+  </material>
   <!-- link mass [kg] -->
   <!-- CURRENTLY ESIMATES - NEED DATA FROM KAWASAKI -->
@@ -13,10 +22,10 @@
   <xacro:property name="pushcorp_mass" value="30"/>
   <!-- joint limits [rad] -->
-  <xacro:property name="j1_lower_limit" value="${radians( 0 )}"/>
-  <xacro:property name="j1_upper_limit" value="${radians( 90 )}"/>
-  <xacro:property name="j2_lower_limit" value="${radians(-80 )}"/>
-  <xacro:property name="j2_upper_limit" value="${radians( 36 )}"/>
-  <xacro:property name="j3_lower_limit" value="${radians(-75 )}"/>
-  <xacro:property name="j3_upper_limit" value="${radians( 0 )}"/>
+  <xacro:property name="j1_lower_limit" value="${radians(-90)}"/>
+  <xacro:property name="j1_upper_limit" value="${radians( 0)}"/>
+  <xacro:property name="j2_lower_limit" value="${radians(-60)}"/>
+  <xacro:property name="j2_upper_limit" value="${radians( 80)}"/>
+  <xacro:property name="j3_lower_limit" value="${radians(-75)}"/>
+  <xacro:property name="j3_upper_limit" value="${radians( 95)}"/>
   <xacro:property name="j4_lower_limit" value="${radians(-210)}"/>
   <xacro:property name="j4_upper_limit" value="${radians( 210)}"/>
@@ -32,133 +41,133 @@
   <xacro:property name="j5_velocity_limit" value="${radians(180)}"/>
   <xacro:property name="j6_velocity_limit" value="${radians(280)}"/>
-  <link name="base_link">
-    <visual>
-      <origin xyz="0 0 0" rpy="0 0 0"/>
-      <geometry>
-        <mesh filename="package://khi2cpp_hw_description/cx110l/meshes/visual/cx165l-base.dae"/>
-      </geometry>
-      <material
-        name="">
-        <color rgba="0.75294 0.75294 0.75294 1" />
-      </material>
-    </visual>
-    <collision>
-      <origin xyz="0 0 0" rpy="0 0 0"/>
-      <geometry>
-        <mesh filename="package://khi2cpp_hw_description/cx110l/meshes/collision/cx165l-base.stl"/>
+  <link name="${prefix}base_link">
+    <visual>
+      <origin xyz="0 0 0" rpy="0 0 0"/>
+      <geometry>
+        <mesh filename="package://khi2cpp_hw_description/cx165l/meshes/visual/cx165l-base.dae"/>
+      </geometry>
+      <material
+        name="">
+        <color rgba="0.75294 0.75294 0.75294 1" />
+      </material>
+    </visual>
+    <collision>
+      <origin xyz="0 0 0" rpy="0 0 0"/>
+      <geometry>
+        <mesh filename="package://khi2cpp_hw_description/cx165l/meshes/collision/cx165l-base.stl"/>
       </geometry>
     </collision>
     <xacro:default_inertial mass="${j0_mass}"/>
   </link>
-  <link name="link_1">
-    <visual>
-      <origin xyz="0 0 0" rpy="0 0 0"/>
-      <geometry>
-        <mesh filename="package://khi2cpp_hw_description/cx110l/meshes/visual/cx165l-j1.dae"/>
-      </geometry>
-      <material
-        name="">
-        <color rgba="0.75294 0.75294 0.75294 1" />
-      </material>
-    </visual>
-    <collision>
-      <origin xyz="0 0 0" rpy="0 0 0"/>
-      <geometry>
-        <mesh filename="package://khi2cpp_hw_description/cx110l/meshes/collision/cx165l-j1.stl"/>
+  <link name="${prefix}link1">
+    <visual>
+      <origin xyz="0 0 0" rpy="0 0 0"/>
+      <geometry>
+        <mesh filename="package://khi2cpp_hw_description/cx165l/meshes/visual/cx165l-j1.dae"/>
+      </geometry>
+      <material
+        name="">
+        <color rgba="0.75294 0.75294 0.75294 1" />
+      </material>
+    </visual>
+    <collision>
+      <origin xyz="0 0 0" rpy="0 0 0"/>
+      <geometry>
+        <mesh filename="package://khi2cpp_hw_description/cx165l/meshes/collision/cx165l-j1.stl"/>
       </geometry>
     </collision>
     <xacro:default_inertial mass="${j1_mass}"/>
   </link>
-  <link name="link_2">
-    <visual>
-      <origin xyz="0 0 0" rpy="0 0 0"/>
-      <geometry>
-        <mesh filename="package://khi2cpp_hw_description/cx110l/meshes/visual/cx165l-j2.dae"/>
-      </geometry>
-      <material
-        name="">
-        <color rgba="0.75294 0.75294 0.75294 1" />
-      </material>
-    </visual>
-    <collision>
-      <origin xyz="0 0 0" rpy="0 0 0"/>
-      <geometry>
-        <mesh filename="package://khi2cpp_hw_description/cx110l/meshes/collision/cx165l-j2.stl"/>
+  <link name="${prefix}link2">
+    <visual>
+      <origin xyz="0 0 0" rpy="0 0 0"/>
+      <geometry>
+        <mesh filename="package://khi2cpp_hw_description/cx165l/meshes/visual/cx165l-j2.dae"/>
+      </geometry>
+      <material
+        name="">
+        <color rgba="0.75294 0.75294 0.75294 1" />
+      </material>
+    </visual>
+    <collision>
+      <origin xyz="0 0 0" rpy="0 0 0"/>
+      <geometry>
+        <mesh filename="package://khi2cpp_hw_description/cx165l/meshes/collision/cx165l-j2.stl"/>
       </geometry>
     </collision>
     <xacro:default_inertial mass="${j2_mass}"/>
   </link>
-  <link name="link_3">
-    <visual>
-      <origin xyz="0 0 0" rpy="0 0 0"/>
-      <geometry>
-        <mesh filename="package://khi2cpp_hw_description/cx110l/meshes/visual/cx165l-j3.dae"/>
-      </geometry>
-      <material
-        name="">
-        <color rgba="0.75294 0.75294 0.75294 1" />
-      </material>
-    </visual>
-    <collision>
-      <origin xyz="0 0 0" rpy="0 0 0"/>
-      <geometry>
-        <mesh filename="package://khi2cpp_hw_description/cx110l/meshes/collision/cx165l-j3.stl"/>
+  <link name="${prefix}link3">
+    <visual>
+      <origin xyz="0 0 0" rpy="0 0 0"/>
+      <geometry>
+        <mesh filename="package://khi2cpp_hw_description/cx165l/meshes/visual/cx165l-j3.dae"/>
+      </geometry>
+      <material
+        name="">
+        <color rgba="0.75294 0.75294 0.75294 1" />
+      </material>
+    </visual>
+    <collision>
+      <origin xyz="0 0 0" rpy="0 0 0"/>
+      <geometry>
+        <mesh filename="package://khi2cpp_hw_description/cx165l/meshes/collision/cx165l-j3.stl"/>
       </geometry>
     </collision>
     <xacro:default_inertial mass="${j3_mass}"/>
   </link>
-  <link name="link_4">
-    <visual>
-      <origin xyz="0 0 0" rpy="0 0 0"/>
-      <geometry>
-        <mesh filename="package://khi2cpp_hw_description/cx110l/meshes/visual/cx165l-j4.dae"/>
-      </geometry>
-      <material
-        name="">
-        <color rgba="0.75294 0.75294 0.75294 1" />
-      </material>
-    </visual>
-    <collision>
-      <origin xyz="0 0 0" rpy="0 0 0"/>
-      <geometry>
-        <mesh filename="package://khi2cpp_hw_description/cx110l/meshes/collision/cx165l-j4.stl"/>
+  <link name="${prefix}link4">
+    <visual>
+      <origin xyz="0 0 0" rpy="0 0 0"/>
+      <geometry>
+        <mesh filename="package://khi2cpp_hw_description/cx165l/meshes/visual/cx165l-j4.dae"/>
+      </geometry>
+      <material
+        name="">
+        <color rgba="0.75294 0.75294 0.75294 1" />
+      </material>
+    </visual>
+    <collision>
+      <origin xyz="0 0 0" rpy="0 0 0"/>
+      <geometry>
+        <mesh filename="package://khi2cpp_hw_description/cx165l/meshes/collision/cx165l-j4.stl"/>
       </geometry>
     </collision>
     <xacro:default_inertial mass="${j4_mass}"/>
   </link>
-  <link name="link_5">
-    <visual>
-      <origin xyz="0 0 0" rpy="0 0 0"/>
-      <geometry>
-        <mesh filename="package://khi2cpp_hw_description/cx110l/meshes/visual/cx165l-j5.dae"/>
-      </geometry>
-      <material
-        name="">
-        <color rgba="0.75294 0.75294 0.75294 1" />
-      </material>
-    </visual>
-    <collision>
-      <origin xyz="0 0 0" rpy="0 0 0"/>
-      <geometry>
-        <mesh filename="package://khi2cpp_hw_description/cx110l/meshes/collision/cx165l-j5.stl"/>
+  <link name="${prefix}link5">
+    <visual>
+      <origin xyz="0 0 0" rpy="0 0 0"/>
+      <geometry>
+        <mesh filename="package://khi2cpp_hw_description/cx165l/meshes/visual/cx165l-j5.dae"/>
+      </geometry>
+      <material
+        name="">
+        <color rgba="0.75294 0.75294 0.75294 1" />
+      </material>
+    </visual>
+    <collision>
+      <origin xyz="0 0 0" rpy="0 0 0"/>
+      <geometry>
+        <mesh filename="package://khi2cpp_hw_description/cx165l/meshes/collision/cx165l-j5.stl"/>
       </geometry>
     </collision>
     <xacro:default_inertial mass="${j5_mass}"/>
   </link>
-  <link name="link_6">
-    <visual>
-      <origin xyz="0 0 0" rpy="0 0 0"/>
-      <geometry>
-        <mesh filename="package://khi2cpp_hw_description/cx110l/meshes/visual/cx165l-j6.dae"/>
-      </geometry>
-      <material
-        name="">
-        <color rgba="0.75294 0.75294 0.75294 1" />
-      </material>
-    </visual>
-    <collision>
-      <origin xyz="0 0 0" rpy="0 0 0"/>
-      <geometry>
-        <mesh filename="package://khi2cpp_hw_description/cx110l/meshes/collision/cx165l-j6.stl"/>
+  <link name="${prefix}link6">
+    <visual>
+      <origin xyz="0 0 0" rpy="0 0 0"/>
+      <geometry>
+        <mesh filename="package://khi2cpp_hw_description/cx165l/meshes/visual/cx165l-j6.dae"/>
+      </geometry>
+      <material
+        name="">
+        <color rgba="0.75294 0.75294 0.75294 1" />
+      </material>
+    </visual>
+    <collision>
+      <origin xyz="0 0 0" rpy="0 0 0"/>
+      <geometry>
+        <mesh filename="package://khi2cpp_hw_description/cx165l/meshes/collision/cx165l-j6.stl"/>
       </geometry>
     </collision>
@@ -169,15 +178,15 @@
       <origin xyz="0 0 0" rpy="0 0 0"/>
       <geometry>
-        <mesh filename="package://khi2cpp_hw_description/cx110l/meshes/visual/cx165l-pushcorp.dae"/>
-      </geometry>
-      <material
-        name="">
-        <color rgba="0.75294 0.75294 0.75294 1" />
-      </material>
-    </visual>
-    <collision>
-      <origin xyz="0 0 0" rpy="0 0 0"/>
-      <geometry>
-        <mesh filename="package://khi2cpp_hw_description/cx110l/meshes/collision/cx165l-pushcorp.stl"/>
+        <mesh filename="package://khi2cpp_hw_description/cx165l/meshes/visual/cx165l-pushcorp.dae"/>
+      </geometry>
+      <material
+        name="">
+        <color rgba="0.75294 0.75294 0.75294 1" />
+      </material>
+    </visual>
+    <collision>
+      <origin xyz="0 0 0" rpy="0 0 0"/>
+      <geometry>
+        <mesh filename="package://khi2cpp_hw_description/cx165l/meshes/collision/cx165l-pushcorp.stl"/>
       </geometry>
     </collision>
@@ -188,58 +197,58 @@
   <joint name="base_joint" type="fixed">
     <parent link="world"/>
-    <child link="base_link"/>
-    <origin xyz="-5.0546 0 0.0254" rpy="0 0 0"/>
+    <child link="${prefix}base_link"/>
+    <origin xyz="0 0 0.0254" rpy="0 0 0"/>
     <axis xyz="0 0 -1"/>
   </joint>
   <!-- joints - main serial chain -->
-  <joint name="joint_1" type="revolute">
-    <parent link="base_link"/>
-    <child link="link_1"/>
+  <joint name="${prefix}joint1" type="revolute">
+    <parent link="${prefix}base_link"/>
+    <child link="${prefix}link1"/>
     <origin xyz="0 0 0.55" rpy="0 0 0"/>
     <axis xyz="0 0 -1"/>
     <limit effort="1000.0" lower="${j1_lower_limit}" upper="${j1_upper_limit}" velocity="${j1_velocity_limit}"/>
   </joint>
-  <joint name="joint_2" type="revolute">
-    <parent link="link_1"/>
-    <child link="link_2"/>
+  <joint name="${prefix}joint2" type="revolute">
+    <parent link="${prefix}link1"/>
+    <child link="${prefix}link2"/>
     <origin xyz="0 0.3 0" rpy="0 0 0"/>
     <axis xyz="1 0 0"/>
     <limit effort="1000.0" lower="${j2_lower_limit}" upper="${j2_upper_limit}" velocity="${j2_velocity_limit}"/>
   </joint>
-  <joint name="joint_3" type="revolute">
-    <parent link="link_2"/>
-    <child link="link_3"/>
+  <joint name="${prefix}joint3" type="revolute">
+    <parent link="${prefix}link2"/>
+    <child link="${prefix}link3"/>
     <origin xyz="0 0 1.19" rpy="0 0 0" />
     <axis xyz="1 0 0"/>
     <limit effort="1000.0" lower="${j3_lower_limit}" upper="${j3_upper_limit}" velocity="${j3_velocity_limit}"/>
   </joint>
-  <joint name="joint_4" type="revolute">
-    <parent link="link_3"/>
-    <child link="link_4"/>
+  <joint name="${prefix}joint4" type="revolute">
+    <parent link="${prefix}link3"/>
+    <child link="${prefix}link4"/>
     <origin xyz="0 1.19 0.3" rpy="0 0 0" />
     <axis xyz="0 1 0"/>
     <limit effort="1000.0" lower="${j4_lower_limit}" upper="${j4_upper_limit}" velocity="${j4_velocity_limit}"/>
   </joint>
-  <joint name="joint_5" type="revolute">
-    <parent link="link_4"/>
-    <child link="link_5"/>
+  <joint name="${prefix}joint5" type="revolute">
+    <parent link="${prefix}link4"/>
+    <child link="${prefix}link5"/>
     <origin xyz="0 0 0" rpy="0 0 0"/>
     <axis xyz="1 0 0"/>
     <limit effort="1000.0" lower="${j5_lower_limit}" upper="${j5_upper_limit}" velocity="${j5_velocity_limit}"/>
   </joint>
-  <joint name="joint_6" type="revolute">
-    <parent link="link_5"/>
-    <child link="link_6"/>
+  <joint name="${prefix}joint6" type="revolute">
+    <parent link="${prefix}link5"/>
+    <child link="${prefix}link6"/>
     <origin xyz="0 0.235 0" rpy="0 0 0" />
     <axis xyz="0 1 0"/>
     <limit effort="1000.0" lower="${j6_lower_limit}" upper="${j6_upper_limit}" velocity="${j6_velocity_limit}"/>
   </joint>
-  <joint name="pushcorp" type="fixed">
-    <parent link="link_6"/>
-    <child link="pushcorp"/>
+  <joint name="${prefix}pushcorp" type="fixed">
+    <parent link="${prefix}link6"/>
+    <child link="${prefix}pushcorp"/>
       <origin xyz="0 0.0949325000000025 0" rpy="0 1.5707963267949 0" />
   </joint>
-  <joint name="joint-tool" type="fixed">
-    <parent link="pushcorp"/>
+  <joint name="${prefix}joint-tool" type="fixed">
+    <parent link="${prefix}pushcorp"/>
     <child link="tool0"/>
     <origin xyz="0 0 .185" rpy="0 0 0"/>

File: ros2_control/cx110l.ros2_control.xacro (robot description, xacro)
@@ -1,18 +1,24 @@
 <?xml version="1.0"?>
 <robot xmlns:xacro="http://www.ros.org/wiki/xacro">
-  <xacro:macro name="cx110l_ros2_control" params="name">
+  <xacro:macro name="cx110l_ros2_control" params="name prefix sim:=true">
     <ros2_control name="${name}" type="system">
       <hardware>
-        <plugin>khi2cpp_hw/KhiSystem</plugin>
-        <param name="ip_address_0">192</param>
-        <param name="ip_address_1">168</param>
-        <param name="ip_address_2">0</param>
-        <param name="ip_address_3">2</param>
-        <param name="period">2</param>
+        <xacro:if value="${sim}">
+          <plugin>mock_components/GenericSystem</plugin>
+        </xacro:if>
+        <xacro:unless value="${sim}">
+          <plugin>khi2cpp_hw/KhiSystem</plugin>
+          <param name="ip_address_0">192</param>
+          <param name="ip_address_1">168</param>
+          <param name="ip_address_2">0</param>
+          <param name="ip_address_3">2</param>
+          <param name="period">2</param>
+          <param name="digital_outputs">1,2</param>
+        </xacro:unless>
       </hardware>
-      <joint name="joint_1">
+      <joint name="${prefix}joint1">
         <command_interface name="position">
-          <param name="min">${radians(0)}</param>
-          <param name="max">${radians(90)}</param>
+          <param name="min">${radians(-160)}</param>
+          <param name="max">${radians(160)}</param>
         </command_interface>
         <command_interface name="velocity">
@@ -20,13 +26,14 @@
           <param name="max">${radians(130)}</param>
         </command_interface>
-        <state_interface name="position">
-          <param name="initial_value">0.0</param>
-        </state_interface>
+        <!-- <command_interface name="acceleration"/> -->
+        <state_interface name="position"/>
         <state_interface name="velocity"/>
+        <param name="initial_position">0.0</param>
+        <param name="initial_velocity">0.0</param>
       </joint>
-      <joint name="joint_2">
+      <joint name="${prefix}joint2">
         <command_interface name="position">
-          <param name="min">${radians(-80)}</param>
-          <param name="max">${radians(36)}</param>
+          <param name="min">${radians(-60)}</param>
+          <param name="max">${radians(80)}</param>
         </command_interface>
         <command_interface name="velocity">
@@ -34,13 +41,14 @@
           <param name="max">${radians(125)}</param>
         </command_interface>
-        <state_interface name="position">
-          <param name="initial_value">0.0</param>
-        </state_interface>
+        <!-- <command_interface name="acceleration"/> -->
+        <state_interface name="position"/>
         <state_interface name="velocity"/>
+        <param name="initial_position">0.0</param>
+        <param name="initial_velocity">0.0</param>
       </joint>
-      <joint name="joint_3">
+      <joint name="${prefix}joint3">
         <command_interface name="position">
           <param name="min">${radians(-75)}</param>
-          <param name="max">${radians(0)}</param>
+          <param name="max">${radians(95)}</param>
         </command_interface>
         <command_interface name="velocity">
@@ -48,10 +56,11 @@
           <param name="max">${radians(125)}</param>
         </command_interface>
-        <state_interface name="position">
-          <param name="initial_value">0.0</param>
-        </state_interface>
+        <!-- <command_interface name="acceleration"/> -->
+        <state_interface name="position"/>
         <state_interface name="velocity"/>
+        <param name="initial_position">${0.0}</param>
+        <param name="initial_velocity">0.0</param>
       </joint>
-      <joint name="joint_4">
+      <joint name="${prefix}joint4">
         <command_interface name="position">
           <param name="min">${radians(-210)}</param>
@@ -62,10 +71,11 @@
           <param name="max">${radians(180)}</param>
         </command_interface>
-        <state_interface name="position">
-          <param name="initial_value">0.0</param>
-        </state_interface>
+        <!-- <command_interface name="acceleration"/> -->
+        <state_interface name="position"/>
         <state_interface name="velocity"/>
+        <param name="initial_position">0.0</param>
+        <param name="initial_velocity">0.0</param>
       </joint>
-      <joint name="joint_5">
+      <joint name="${prefix}joint5">
         <command_interface name="position">
           <param name="min">${radians(-120)}</param>
@@ -76,10 +86,11 @@
           <param name="max">${radians(180)}</param>
         </command_interface>
-        <state_interface name="position">
-          <param name="initial_value">0.0</param>
-        </state_interface>
+        <!-- <command_interface name="acceleration"/> -->
+        <state_interface name="position"/>
         <state_interface name="velocity"/>
+        <param name="initial_position">0.0</param>
+        <param name="initial_velocity">0.0</param>
       </joint>
-      <joint name="joint_6">
+      <joint name="${prefix}joint6">
         <command_interface name="position">
           <param name="min">${radians(-360)}</param>
@@ -90,8 +101,9 @@
           <param name="max">${radians(280)}</param>
         </command_interface>
-        <state_interface name="position">
-          <param name="initial_value">0.0</param>
-        </state_interface>
+        <!-- <command_interface name="acceleration"/> -->
+        <state_interface name="position"/>
         <state_interface name="velocity"/>
+        <param name="initial_position">1.571</param>
+        <param name="initial_velocity">0.0</param>
       </joint>
     </ros2_control>
