Commit message: Updated components of driver

File: ros2_control/cx165l.ros2_control.xacro (robot description, xacro)
@@ -4,4 +4,8 @@
     <ros2_control name="${name}" type="system">
       <hardware>
+        <xacro:if value="${sim}">
+          <plugin>mock_components/GenericSystem</plugin>
+        </xacro:if>
+        <xacro:unless value="${sim}">
         <plugin>khi2cpp_hw/KhiSystem</plugin>
         <param name="ip_address_0">192</param>
@@ -10,6 +14,7 @@
         <param name="ip_address_3">23</param>
         <param name="period">2</param>
+        </xacro:unless>
       </hardware>
-      <joint name="joint_1">
+      <joint name="${prefix}joint1">
         <command_interface name="position">
           <param name="min">${radians(-160)}</param>
@@ -20,10 +25,11 @@
           <param name="max">${radians(130)}</param>
         </command_interface>
-        <state_interface name="position">
-          <param name="initial_value">0.0</param>
-        </state_interface>
+        <!-- <command_interface name="acceleration"/> -->
+        <state_interface name="position"/>
         <state_interface name="velocity"/>
+        <param name="initial_position">0.0</param>
+        <param name="initial_velocity">0.0</param>
       </joint>
-      <joint name="joint_2">
+      <joint name="${prefix}joint2">
         <command_interface name="position">
           <param name="min">${radians(-60)}</param>
@@ -34,10 +40,11 @@
           <param name="max">${radians(125)}</param>
         </command_interface>
-        <state_interface name="position">
-          <param name="initial_value">0.0</param>
-        </state_interface>
+        <!-- <command_interface name="acceleration"/> -->
+        <state_interface name="position"/>
         <state_interface name="velocity"/>
+        <param name="initial_position">0.0</param>
+        <param name="initial_velocity">0.0</param>
       </joint>
-      <joint name="joint_3">
+      <joint name="${prefix}joint3">
         <command_interface name="position">
           <param name="min">${radians(-75)}</param>
@@ -48,10 +55,11 @@
           <param name="max">${radians(125)}</param>
         </command_interface>
-        <state_interface name="position">
-          <param name="initial_value">0.0</param>
-        </state_interface>
+        <!-- <command_interface name="acceleration"/> -->
+        <state_interface name="position"/>
         <state_interface name="velocity"/>
+        <param name="initial_position">${0.0}</param>
+        <param name="initial_velocity">0.0</param>
       </joint>
-      <joint name="joint_4">
+      <joint name="${prefix}joint4">
         <command_interface name="position">
           <param name="min">${radians(-210)}</param>
@@ -62,10 +70,11 @@
           <param name="max">${radians(180)}</param>
         </command_interface>
-        <state_interface name="position">
-          <param name="initial_value">0.0</param>
-        </state_interface>
+        <!-- <command_interface name="acceleration"/> -->
+        <state_interface name="position"/>
         <state_interface name="velocity"/>
+        <param name="initial_position">0.0</param>
+        <param name="initial_velocity">0.0</param>
       </joint>
-      <joint name="joint_5">
+      <joint name="${prefix}joint5">
         <command_interface name="position">
           <param name="min">${radians(-120)}</param>
@@ -76,10 +85,11 @@
           <param name="max">${radians(180)}</param>
         </command_interface>
-        <state_interface name="position">
-          <param name="initial_value">0.0</param>
-        </state_interface>
+        <!-- <command_interface name="acceleration"/> -->
+        <state_interface name="position"/>
         <state_interface name="velocity"/>
+        <param name="initial_position">0.0</param>
+        <param name="initial_velocity">0.0</param>
       </joint>
-      <joint name="joint_6">
+      <joint name="${prefix}joint6">
         <command_interface name="position">
           <param name="min">${radians(-360)}</param>
@@ -90,8 +100,9 @@
           <param name="max">${radians(280)}</param>
         </command_interface>
-        <state_interface name="position">
-          <param name="initial_value">0.0</param>
-        </state_interface>
+        <!-- <command_interface name="acceleration"/> -->
+        <state_interface name="position"/>
         <state_interface name="velocity"/>
+        <param name="initial_position">1.571</param>
+        <param name="initial_velocity">0.0</param>
       </joint>
     </ros2_control>

Commit message: updates

File: cx110l/urdf/cx110l_macro.xacro (robot description, xacro)
@@ -218,5 +218,5 @@
     <child link="${prefix}link1"/>
     <origin xyz="0 0 0.55" rpy="0 0 0"/>
-    <axis xyz="0 0 -1"/>
+    <axis xyz="0 0 -1" rpy="0 0 0" />
     <limit effort="1000.0" lower="${j1_lower_limit}" upper="${j1_upper_limit}" velocity="${j1_velocity_limit}"/>
   </joint>
@@ -224,6 +224,6 @@
     <parent link="${prefix}link1"/>
     <child link="${prefix}link2"/>
-    <origin xyz="0 0.3 0" rpy="0 0 0"/>
-    <axis xyz="1 0 0"/>
+    <origin xyz="0.3 0.0 0" rpy="0 0 0" />
+    <axis xyz="0 1 0" rpy="0 0 0" />
     <limit effort="1000.0" lower="${j2_lower_limit}" upper="${j2_upper_limit}" velocity="${j2_velocity_limit}"/>
   </joint>
@@ -232,5 +232,5 @@
     <child link="${prefix}link3"/>
     <origin xyz="0 0 1.19" rpy="0 0 0" />
-    <axis xyz="1 0 0"/>
+    <axis xyz="0 -1 0" rpy="0 0 0" />
     <limit effort="1000.0" lower="${j3_lower_limit}" upper="${j3_upper_limit}" velocity="${j3_velocity_limit}"/>
   </joint>

File: cx165l/urdf/cx165l_macro.xacro (robot description, xacro)
@@ -41,4 +41,12 @@
   <xacro:property name="j5_velocity_limit" value="${radians(180)}"/>
   <xacro:property name="j6_velocity_limit" value="${radians(280)}"/>
+  <!-- link inertial(TODO : set correct link inertial )-->
+  <xacro:macro name="default_inertial" params="mass">
+    <inertial>
+      <mass value="${mass}" />
+      <inertia ixx="0.1" ixy="0.0" ixz="0.0" iyy="0.1" iyz="0.0" izz="0.1" />
+    </inertial>
+  </xacro:macro>
+  <link name="world"/>
   <link name="${prefix}base_link">
     <visual>
@@ -205,6 +213,6 @@
     <parent link="${prefix}base_link"/>
     <child link="${prefix}link1"/>
-    <origin xyz="0 0 0.55" rpy="0 0 0"/>
-    <axis xyz="0 0 -1"/>
+    <origin xyz="0 0 0.55" rpy="0 0 0" />
+    <axis xyz="0 0 -1" rpy="0 0 0" />
     <limit effort="1000.0" lower="${j1_lower_limit}" upper="${j1_upper_limit}" velocity="${j1_velocity_limit}"/>
   </joint>
@@ -213,5 +221,5 @@
     <child link="${prefix}link2"/>
     <origin xyz="0 0.3 0" rpy="0 0 0"/>
-    <axis xyz="1 0 0"/>
+    <axis xyz="0 1 0" rpy="0 0 0" />
     <limit effort="1000.0" lower="${j2_lower_limit}" upper="${j2_upper_limit}" velocity="${j2_velocity_limit}"/>
   </joint>
@@ -220,5 +228,5 @@
     <child link="${prefix}link3"/>
     <origin xyz="0 0 1.19" rpy="0 0 0" />
-    <axis xyz="1 0 0"/>
+    <axis xyz="0 -1 0" rpy="0 0 0" />
     <limit effort="1000.0" lower="${j3_lower_limit}" upper="${j3_upper_limit}" velocity="${j3_velocity_limit}"/>
   </joint>
@@ -233,6 +241,6 @@
     <parent link="${prefix}link4"/>
     <child link="${prefix}link5"/>
-    <origin xyz="0 0 0" rpy="0 0 0"/>
-    <axis xyz="1 0 0"/>
+    <origin rpy="0 0 0" xyz="0 0 0"/>
+    <axis xyz="0 -1 0" rpy="0 0 0" />
     <limit effort="1000.0" lower="${j5_lower_limit}" upper="${j5_upper_limit}" velocity="${j5_velocity_limit}"/>
   </joint>
@@ -247,10 +255,10 @@
     <parent link="${prefix}link6"/>
     <child link="${prefix}pushcorp"/>
-      <origin xyz="0 0.0949325000000025 0" rpy="0 1.5707963267949 0" />
+      <origin xyz="0 0.0949325000000025 0" rpy="0 0 0" />
   </joint>
   <joint name="${prefix}joint-tool" type="fixed">
     <parent link="${prefix}pushcorp"/>
     <child link="tool0"/>
-    <origin xyz="0 0 .185" rpy="0 0 0"/>
+    <origin xyz="0.3567 0.15 0" rpy="0 0 0"/>
   </joint>
 </xacro:macro>

File: cx165l/urdf/workcell.xacro (robot description, xacro)
@@ -3,13 +3,12 @@
   <!-- <xacro:property name="robot_name" value="cx165l"/>
   <xacro:property name="krnx_name" value="CX165L-BC01"/> -->
-  <xacro:khi_cx165l prefix="" />
+  <xacro:arg name="prefix" default=""/>
+  <!-- Import Lab Robot Cell -->
+  <xacro:include filename="$(find khi2cpp_hw_description)/common/isu_lab.xacro" />
   <!-- Import cx165l macro -->
   <xacro:include filename="$(find khi2cpp_hw_description)/cx165l/urdf/cx165l_macro.xacro"/>
-  <!-- create link fixed to the "world" -->
-  <link name="world"/>
-  <!-- Import Lab Robot Cell -->
-  <xacro:include filename="$(find khi2cpp_hw_description)/common/isu_lab.xacro" />
-  <xacro:cx165l_description/>
-  <!-- Import cx110l ros2_control description -->
+  <xacro:khi_cx165l prefix="" />
+  <xacro:arg name="sim" default="false"/>
+  <!-- Import cx165l ros2_control description -->
   <xacro:include filename="$(find khi2cpp_hw_description)/ros2_control/cx165l.ros2_control.xacro" />
   <xacro:cx165l_ros2_control name="CX165L-BC01" prefix="" sim="$(arg sim)"/>

File: ros2_control/cx110l.ros2_control.xacro (robot description, xacro)
@@ -1,5 +1,5 @@
 <?xml version="1.0"?>
 <robot xmlns:xacro="http://www.ros.org/wiki/xacro">
-  <xacro:macro name="cx110l_ros2_control" params="name prefix sim:=true">
+  <xacro:macro name="cx165l_ros2_control" params="name prefix sim:=true">
     <ros2_control name="${name}" type="system">
       <hardware>

File: ros2_control/cx165l.ros2_control.xacro (robot description, xacro)
@@ -1,5 +1,5 @@
 <?xml version="1.0"?>
 <robot xmlns:xacro="http://www.ros.org/wiki/xacro">
-  <xacro:macro name="cx165l_ros2_control" params="name">
+  <xacro:macro name="cx165l_ros2_control" params="name prefix sim:=true">
     <ros2_control name="${name}" type="system">
       <hardware>
@@ -14,4 +14,5 @@
         <param name="ip_address_3">23</param>
         <param name="period">2</param>
+        <param name="digital_outputs">1,2</param>
         </xacro:unless>
       </hardware>
